Commit message: fix: adjusted visual now included

File: src/quad_navigation/urdf/geometry.urdf.xacro (robot description, xacro)
@@ -1,4 +1,6 @@
 <?xml version="1.0"?>
-<robot name="drone">
+<robot xmlns:xacro="http://www.ros.org/wiki/xacro" name="drone">
+    <xacro:property name="length" value="0.2"/>
+    <xacro:property name="radius" value="0.2"/>
     <link name="body_link">
         <visual>
@@ -16,5 +18,5 @@
         <visual>
             <geometry>
-                <cylinder length="0.2" radius="0.2"/>
+                <cylinder length="${length}" radius="${radius}"/>
             </geometry>
             <!-- <material name="orange"/> -->
@@ -22,5 +24,5 @@
         <collision>
             <geometry>
-                <cylinder length="0.2" radius="0.2"/>
+                <cylinder length="${length}" radius="${radius}"/>
             </geometry>
         </collision>
@@ -29,5 +31,5 @@
         <visual>
             <geometry>
-                <cylinder length="0.2" radius="0.2"/>
+                <cylinder length="${length}" radius="${radius}"/>
             </geometry>
             <!-- <material name="orange"/> -->
@@ -35,5 +37,5 @@
         <collision>
             <geometry>
-                <cylinder length="0.2" radius="0.2"/>
+                <cylinder length="${length}" radius="${radius}"/>
             </geometry>
         </collision>
@@ -42,10 +44,10 @@
         <visual>
             <geometry>
-                <cylinder length="0.2" radius="0.2"/>
+                <cylinder length="${length}" radius="${radius}"/>
             </geometry>
         </visual>
         <collision>
             <geometry>
-                <cylinder length="0.2" radius="0.2"/>
+                <cylinder length="${length}" radius="${radius}"/>
             </geometry>
         </collision>
@@ -54,10 +56,10 @@
         <visual>
             <geometry>
-                <cylinder length="0.2" radius="0.2"/>
+                <cylinder length="${length}" radius="${radius}"/>
             </geometry>
         </visual>
         <collision>
             <geometry>
-                <cylinder length="0.2" radius="0.2"/>
+                <cylinder length="${length}" radius="${radius}"/>
             </geometry>
         </collision>
